File: pcb/IC_PCB_v2/IC_PCB_v2.kicad_pcb (KiCad board)
At the start: 2 copper layers, 30 x 27.4 mm, 17 parts, among them IC1 MAX30102EFD+, IC2 MAX30205MTA+, J1 52207-0460, U1 AZ1084-1.8

Commit message: uploaded code and stuff
Parts:
- removed U1: AZ1084-1.8, Package_TO_SOT_SMD:TO-252-3_TabPin2
- added U2: ADP7182AUJZ-1.8, Package_TO_SOT_SMD:TSOT-23-5, F.Cu at (138.5, 77.7)
- C1: value 10u -> 2u2; footprint Capacitor_SMD:C_1206_3216Metric -> Capacitor_SMD:C_0603_1608Metric
- C2: value 22u -> 2u2; footprint Capacitor_SMD:C_1206_3216Metric -> Capacitor_SMD:C_0603_1608Metric
- C3, C7: footprint Capacitor_SMD:C_0201_0603Metric_Pad0.64x0.40mm_HandSolder -> Capacitor_SMD:C_0603_1608Metric
- moved C1 10.2 mm to (135.0, 78.1), turned to 135 degrees
- moved C2 3.03 mm to (142.1, 78.7), turned to 45 degrees
- moved C5 0.82 mm to (150.9, 91.9)
- moved C9 0.82 mm to (146.4, 89.5)
- moved C3 0.80 mm to (149.4, 92.5)
- moved C7 0.56 mm to (147.8, 89.8)
Routing:
- net +3V3: track 55.3 -> 75.5 mm
- net GND: track 26.2 -> 27.9 mm, vias 67 -> 37
Other:
- board size 30 x 27.4 mm -> 30 x 21.4 mm
- board text added: "JLCJLCJLCJLC"
