File: pcb/pulse_ox_wearable/pulse_ox_wearable.kicad_pcb (KiCad board)
At the start: 4 copper layers, 65.6 x 65.6 mm, 45 parts, among them J1 JST Battery In, J2 USB4800-03-A, J3 52207-0460, J4 OLED, Q1 BC817, Q2 BC817, SW1 450302014072, SW2 SW_Push, U1 ESP32-S3-WROOM-2-N32R8V, U2 MCP73832T-2DCI/OT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

Commit message: updated for week 4
Parts:
- moved J4 1.03 mm to (117.3, 72.3)
Routing:
- net ~{CS}: track 0.00 -> 62.0 mm, vias 0 -> 2
- net SCLK: track 0.00 -> 60.9 mm, vias 0 -> 1
- net MOSI: track 0.00 -> 56.0 mm, vias 0 -> 1
- net DC: track 0.00 -> 52.1 mm, vias 0 -> 1
- net RST: track 0.00 -> 49.8 mm, vias 0 -> 1
- net +3V3: track 106.3 -> 147.3 mm
- net GND: track 102.9 -> 85.7 mm, vias 249 -> 186
- net IO0: track 41.4 -> 42.6 mm

Commit message: uploaded code and stuff
Parts:
- moved I2C 1.00 mm to (112.3, 57.8)
- renumbered J3 to I2C
Routing:
- net GND: track 85.7 -> 78.9 mm, vias 186 -> 185
- net +3V3: track 147.3 -> 145.8 mm
- net SCL: track 17.4 -> 15.9 mm
- net SDA: track 22.6 -> 21.6 mm
- net ~{CS}: track 62.0 -> 61.5 mm, vias 2 -> 1
Other:
- board text added: "+"
- board text added: "-"
- board text added: "3V3"
- board text added: "BL"
- board text added: "DC"
- board text added: "GND"
- board text added: "MOSI"
- board text added: "RST"
- board text added: "SCLK"
- board text added: "~{CS}"

Commit message: updating
Parts:
- L1: value XFL4020-102MEB -> TFM322512ALVA1R0MTAA; footprint my_foot:L_SMD_4.8_x_2.85 -> Inductor_SMD:L_1210_3225Metric
- R1, R2: footprint Resistor_SMD:R_0201_0603Metric -> Resistor_SMD:R_0402_1005Metric
- moved L1 0.32 mm to (87.5, 84.2)
- renumbered I2C to J3
