File: pcb/pulse_ox_wearable/pulse_ox_wearable.kicad_sch (KiCad schematic)
At the start: 45 parts, among them J1 JST Battery In, J2 USB4800-03-A, J3 52207-0460, J4 OLED, Q1 BC817, Q2 BC817, SW1 450302014072, SW2 SW_Push, U1 ESP32-S3-WROOM-2-N32R8V, U2 MCP73832T-2DCI/OT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

Commit message: uploaded code and stuff
Changed lines of the file:
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@@
   )
   (text "Truth Table\nDTR RTS -> EN IO0\n 1   1      1   1 \n 0   0      1   1\n 1   0      0   1\n 0   1      1   0 "
-    (at 158.75 71.12 0)
+    (at 158.75 72.39 0)
     (effects (font (size 1.27 1.27)) (justify left bottom))
   )

Commit message: updating
Parts:
- L1: value XFL4020-102MEB -> TFM322512ALVA1R0MTAA; footprint my_foot:L_SMD_4.8_x_2.85 -> Inductor_SMD:L_1210_3225Metric
Changed lines of the file:
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@@
       (effects (font (size 1.27 1.27)))
     )
-    (property "Value" "XFL4020-102MEB" (at 203.2 17.78 90)
-      (effects (font (size 1.27 1.27)))
-    )
-    (property "Footprint" "my_foot:L_SMD_4.8_x_2.85" (at 203.2 20.32 0)
+    (property "Value" "TFM322512ALVA1R0MTAA" (at 203.2 17.78 90)
+      (effects (font (size 1.27 1.27)))
+    )
+    (property "Footprint" "Inductor_SMD:L_1210_3225Metric" (at 203.2 20.32 0)
       (effects (font (size 1.27 1.27)) hide)
     )
@@
   (symbol (lib_id "Connector:Conn_01x04_Female") (at 171.45 115.57 0) (unit 1)
     (in_bom yes) (on_board yes) (dnp no) (fields_autoplaced)
-    (property "Reference" "J3" (at 172.72 115.5699 0)
-      (effects (font (size 1.27 1.27)) (justify left))
-    )
-    (property "Value" "52207-0460 " (at 172.72 118.1099 0)
-      (effects (font (size 1.27 1.27)) (justify left))
-    )
+    (property "Reference" "J3" (at 172.72 115.57 0)
+      (effects (font (size 1.27 1.27)) (justify left))
+    )
+    (property "Value" "52207-0460 " (at 172.72 118.11 0)
+      (effects (font (size 1.27 1.27)) (justify left))
+    )
